File: HARDWARE/ant control board v1.3/ant control board v1.3.kicad_pcb (KiCad board)
At the start: 2 copper layers, 22.8 x 33.2 mm, 97 parts, among them J1 B_SW, J10 M2, J11 M3, J2 2s Battery, J4 USB-C_304A-ACP16X, J5 custom analog 2, J6 custom analog 1, J7 servo 2, J8 servo 1 (HV), J9 M1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

Commit message: fixed the no tank mix problem
without using the tank mix FAC should control individual DC motors directly using the remote controller channel's value, but it did't. Now it does (the error was not passing the enum number)
Parts:
- removed kibuzzard-66CF23DF: G***, kibuzzard-66CF23DF
- added kibuzzard-66A643AC: G***, kibuzzard-66A643AC, B.Cu at (154.3, 71.6)
Changed lines of the file:
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@@
 		)
 	)
+	(footprint "kibuzzard-66A643AC"
+		(layer "B.Cu")
+		(at 154.2796 71.628)
+		(descr "Generated with KiBuzzard")
+		(tags "kb_params=eyJBbGlnbm1lbnRDaG9pY2UiOiAiQ2VudGVyIiwgIkNhcExlZnRDaG9pY2UiOiAiKCIsICJDYXBSaWdodENob2ljZSI6ICIpIiwgIkZvbnRDb21ib0JveCI6ICJFUkFTQkQiLCAiSGVpZ2h0Q3RybCI6IDEuMCwgIkxheWVyQ29tYm9Cb3giOiAiRi5TaWxrUyIsICJMaW5lU3BhY2luZ0N0cmwiOiAxLjUsICJNdWx0aUxpbmVUZXh0IjogIi0gICAgKyIsICJQYWRkaW5nQm90dG9tQ3RybCI6IDEuMCwgIlBhZGRpbmdMZWZ0Q3RybCI6IDkuMCwgIlBhZGRpbmdSaWdodEN0cmwiOiA5LjAsICJQYWRkaW5nVG9wQ3RybCI6IDEuMCwgIldpZHRoQ3RybCI6IDAuMCwgImFkdmFuY2VkQ2hlY2tib3giOiB0cnVlLCAiaW5saW5lRm9ybWF0VGV4dGJveCI6IGZhbHNlLCAibGluZW92ZXJTdHlsZUNob2ljZSI6ICJTcXVhcmUiLCAibGluZW92ZXJUaGlja25lc3NDdHJsIjogOH0=")
+		(property "Reference" "kibuzzard-66A643AC"
+			(at 0 3.595741 0)
+			(layer "B.SilkS")
+			(hide yes)
+			(effects
+				(font
+					(size 0.001 0.001)
+				)
+				(justify mirror)
+			)
+		)
+		(property "Value" "G***"
+			(at 0 -3.595741 0)
+			(layer "B.SilkS")
+			(hide yes)
+			(effects
+				(font
+					(size 0.001 0.001)
+				)
+				(justify mirror)
+			)
+		)
+		(property "Footprint" "kibuzzard-66A643AC"
+			(at 0 0 180)
+			(unlocked yes)
+			(layer "B.Fab")
+			(hide yes)
+			(effects
+				(font
+					(size 1.27 1.27)
+				)
+				(justify mirror)
+			)
+		)
+		(property "Datasheet" ""
+			(at 0 0 180)
+			(unlocked yes)
+			(layer "B.Fab")
+			(hide yes)
+			(effects
+				(font
+					(size 1.27 1.27)
+				)
+				(justify mirror)
+			)
+		)
+		(property "Description" ""
+			(at 0 0 180)
+			(unlocked yes)
+			(layer "B.Fab")
+			(hide yes)
+			(effects
+				(font
+					(size 1.27 1.27)
+				)
+				(justify mirror)
+			)
+		)
+		(attr board_only exclude_from_pos_files exclude_from_bom)
+		(fp_poly
+			(pts
+				(xy -1.412454 0.547741) (xy -2.537729 0.547741) (xy -2.644588 0.537216) (xy -2.74734 0.506047) (xy -2.842038 0.45543)
+				(xy -2.92504 0.387311) (xy -2.993159 0.304309) (xy -3.043776 0.209611) (xy -3.074945 0.106859) (xy -3.08547 0)
+				(xy -3.074945 -0.106859) (xy -3.043776 -0.209611) (xy -2.993159 -0.304309) (xy -2.92504 -0.387311)
+				(xy -2.842038 -0.45543) (xy -2.74734 -0.506047) (xy -2.644588 -0.537216) (xy -2.537729 -0.547741)
+				(xy -1.412454 -0.547741) (xy -1.412454 -0.227106) (xy -1.405311 -0.12326) (xy -1.401465 -0.024176)
+				(xy -1.300366 -0.026374) (xy -1.205128 -0.027106) (xy -1.108974 -0.026374) (xy -1.008059 -0.024176)
+				(xy -1.015202 -0.122161) (xy -1.019048 -0.227106) (xy -1.12033 -0.225458) (xy -1.216117 -0.224908)
+				(xy -1.311722 -0.225458) (xy -1.412454 -0.227106) (xy -1.412454 -0.547741) (xy 1.060073 -0.547741)
+				(xy 1.060073 -0.422711) (xy 0.964835 -0.420513) (xy 0.869597 -0.422711) (xy 0.887912 -0.088645)
+				(xy 0.71282 -0.089377) (xy 0.559707 -0.090842) (xy 0.565751 -0.00641) (xy 0.569231 0.091575) (xy 0.739927 0.09011)
+				(xy 0.897436 0.089377) (xy 0.911355 0.422711) (xy 1.006593 0.421245) (xy 1.101831 0.422711) (xy 1.082784 0.089377)
+				(xy 1.281319 0.09011) (xy 1.412454 0.091575) (xy 1.406776 0.007143) (xy 1.40293 -0.090842) (xy 1.272527 -0.09011)
+				(xy 1.073993 -0.088645) (xy 1.071469 -0.144648) (xy 1.066829 -0.256003) (xy 1.060073 -0.422711)
+				(xy 1.060073 -0.547741) (xy 1.412454 -0.547741) (xy 2.537729 -0.547741) (xy 2.644588 -0.537216)
+				(xy 2.74734 -0.506047) (xy 2.842037 -0.45543) (xy 2.92504 -0.387311) (xy 2.993159 -0.304309) (xy 3.043776 -0.209611)
+				(xy 3.074945 -0.106859) (xy 3.08547 0) (xy 3.074945 0.106859) (xy 3.043776 0.209611) (xy 2.993159 0.304309)
+				(xy 2.92504 0.387311) (xy 2.842037 0.45543) (xy 2.74734 0.506047) (xy 2.644588 0.537216) (xy 2.537729 0.547741)
+				(xy 1.412454 0.547741) (xy -1.412454 0.547741)
+			)
+			(stroke
+				(width 0)
+				(type solid)
+			)
+			(fill solid)
+			(layer "B.SilkS")
+		)
+	)
 	(footprint "Jumper:SolderJumper-3_P1.3mm_Open_RoundedPad1.0x1.5mm_NumberLabels"
 		(layer "B.Cu")
@@
 			)
 			(stroke
-				(width 0)
-				(type solid)
-			)
-			(fill solid)
-			(layer "B.SilkS")
-		)
-	)
-	(footprint "kibuzzard-66CF23DF"
-		(layer "B.Cu")
-		(at 154.2796 71.628)
-		(descr "Generated with KiBuzzard")
-		(tags "kb_params=eyJBbGlnbm1lbnRDaG9pY2UiOiAiQ2VudGVyIiwgIkNhcExlZnRDaG9pY2UiOiAiKCIsICJDYXBSaWdodENob2ljZSI6ICIpIiwgIkZvbnRDb21ib0JveCI6ICJFUkFTQkQiLCAiSGVpZ2h0Q3RybCI6IDEuMCwgIkxheWVyQ29tYm9Cb3giOiAiRi5TaWxrUyIsICJMaW5lU3BhY2luZ0N0cmwiOiAxLjUsICJNdWx0aUxpbmVUZXh0IjogIisgICAgLSIsICJQYWRkaW5nQm90dG9tQ3RybCI6IDEuMCwgIlBhZGRpbmdMZWZ0Q3RybCI6IDkuMCwgIlBhZGRpbmdSaWdodEN0cmwiOiA5LjAsICJQYWRkaW5nVG9wQ3RybCI6IDEuMCwgIldpZHRoQ3RybCI6IDAuMCwgImFkdmFuY2VkQ2hlY2tib3giOiB0cnVlLCAiaW5saW5lRm9ybWF0VGV4dGJveCI6IGZhbHNlLCAibGluZW92ZXJTdHlsZUNob2ljZSI6ICJTcXVhcmUiLCAibGluZW92ZXJUaGlja25lc3NDdHJsIjogOH0=")
-		(property "Reference" "kibuzzard-66CF23DF"
-			(at 0 3.595741 0)
-			(layer "B.SilkS")
-			(hide yes)
-			(effects
-				(font
-					(size 0.001 0.001)
-				)
-				(justify mirror)
-			)
-		)
-		(property "Value" "G***"
-			(at 0 -3.595741 0)
-			(layer "B.SilkS")
-			(hide yes)
-			(effects
-				(font
-					(size 0.001 0.001)
-				)
-				(justify mirror)
-			)
-		)
-		(property "Footprint" "kibuzzard-66CF23DF"
-			(at 0 0 180)
-			(unlocked yes)
-			(layer "B.Fab")
-			(hide yes)
-			(effects
-				(font
-					(size 1.27 1.27)
-				)
-				(justify mirror)
-			)
-		)
-		(property "Datasheet" ""
-			(at 0 0 180)
-			(unlocked yes)
-			(layer "B.Fab")
-			(hide yes)
-			(effects
-				(font
-					(size 1.27 1.27)
-				)
-				(justify mirror)
-			)
-		)
-		(property "Description" ""
-			(at 0 0 180)
-			(unlocked yes)
-			(layer "B.Fab")
-			(hide yes)
-			(effects
-				(font
-					(size 1.27 1.27)
-				)
-				(justify mirror)
-			)
-		)
-		(attr board_only exclude_from_pos_files exclude_from_bom)
-		(fp_poly
-			(pts
-				(xy -1.405495 0.547741) (xy -2.530769 0.547741) (xy -2.637628 0.537216) (xy -2.740381 0.506047)
-				(xy -2.835078 0.45543) (xy -2.918081 0.387311) (xy -2.986199 0.304309) (xy -3.036816 0.209611) (xy -3.067986 0.106859)
-				(xy -3.07851 0) (xy -3.067986 -0.106859) (xy -3.036816 -0.209611) (xy -2.986199 -0.304309) (xy -2.918081 -0.387311)
-				(xy -2.835078 -0.45543) (xy -2.740381 -0.506047) (xy -2.637628 -0.537216) (xy -2.530769 -0.547741)
-				(xy -1.405495 -0.547741) (xy -0.905128 -0.547741) (xy -0.905128 -0.422711) (xy -1.000366 -0.420513)
-				(xy -1.095605 -0.422711) (xy -1.077289 -0.088645) (xy -1.252381 -0.089377) (xy -1.405495 -0.090842)
-				(xy -1.399451 -0.00641) (xy -1.395971 0.091575) (xy -1.225275 0.09011) (xy -1.067766 0.089377) (xy -1.053846 0.422711)
-				(xy -0.958608 0.421245) (xy -0.86337 0.422711) (xy -0.882418 0.089377) (xy -0.683883 0.09011) (xy -0.552747 0.091575)
-				(xy -0.558425 0.007143) (xy -0.562271 -0.090842) (xy -0.692674 -0.09011) (xy -0.891209 -0.088645)
-				(xy -0.893732 -0.144648) (xy -0.898372 -0.256003) (xy -0.905128 -0.422711) (xy -0.905128 -0.547741)
-				(xy 1.001099 -0.547741) (xy 1.001099 -0.227106) (xy 1.008242 -0.12326) (xy 1.012088 -0.024176) (xy 1.113187 -0.026374)
-				(xy 1.208425 -0.027106) (xy 1.304579 -0.026374) (xy 1.405494 -0.024176) (xy 1.398352 -0.122161)
-				(xy 1.394505 -0.227106) (xy 1.293223 -0.225458) (xy 1.197436 -0.224908) (xy 1.101831 -0.225458)
-				(xy 1.001099 -0.227106) (xy 1.001099 -0.547741) (xy 1.405494 -0.547741) (xy 2.530769 -0.547741)
-				(xy 2.637628 -0.537216) (xy 2.740381 -0.506047) (xy 2.835078 -0.45543) (xy 2.918081 -0.387311) (xy 2.986199 -0.304309)
-				(xy 3.036816 -0.209611) (xy 3.067986 -0.106859) (xy 3.07851 0) (xy 3.067986 0.106859) (xy 3.036816 0.209611)
-				(xy 2.986199 0.304309) (xy 2.918081 0.387311) (xy 2.835078 0.45543) (xy 2.740381 0.506047) (xy 2.637628 0.537216)
-				(xy 2.530769 0.547741) (xy 1.405494 0.547741) (xy -1.405495 0.547741)
-			)
-			(stroke
